File: pcb/JJL_PCB/JJL_PCB.kicad_pcb (KiCad board)
At the start: 2 copper layers, 129.5 x 112.2 mm, 28 parts, among them J1 Conn_01x04_Pin, J2 Conn_01x04_Pin, J3 Conn_01x04_Pin, J4 Conn_01x04_Pin, U1 STM32G0B1KCTx, U2 L7805CV-DG, U3 TLV70033_SOT23-5

Commit message: hi
Parts:
- removed C3: 1u, Capacitor_SMD:C_0402_1005Metric_Pad0.74x0.62mm_HandSolder
- removed J2, J3, J4: Conn_01x04_Pin, Connector_PinHeader_2.54mm:PinHeader_1x04_P2.54mm_Vertical
- added TP10: TestPoint, TestPoint:TestPoint_Pad_D3.0mm, F.Cu at (166.0, 171.0)
- added TP11: TestPoint, TestPoint:TestPoint_Pad_D3.0mm, F.Cu at (188.0, 197.0)
- added TP12: TestPoint, TestPoint:TestPoint_Pad_D3.0mm, F.Cu at (219.0, 197.0)
- added TP13: TestPoint, TestPoint:TestPoint_Pad_D3.0mm, F.Cu at (160.0, 178.0)
- added TP14: TestPoint, TestPoint:TestPoint_Pad_D3.0mm, F.Cu at (178.0, 197.0)
- added TP15: TestPoint, TestPoint:TestPoint_Pad_D3.0mm, F.Cu at (231.0, 197.0)
- added TP4: TestPoint, TestPoint:TestPoint_Pad_D3.0mm, F.Cu at (232.0, 146.0)
- added TP5: TestPoint, TestPoint:TestPoint_Pad_D3.0mm, F.Cu at (243.0, 166.0)
- added TP6: TestPoint, TestPoint:TestPoint_Pad_D3.0mm, F.Cu at (187.0, 129.0)
- added TP7: TestPoint, TestPoint:TestPoint_Pad_D3.0mm, F.Cu at (234.0, 162.0)
- added TP8: TestPoint, TestPoint:TestPoint_Pad_D3.0mm, F.Cu at (223.0, 137.0)
- added TP9: TestPoint, TestPoint:TestPoint_Pad_D3.0mm, F.Cu at (180.0, 140.0)
- added U4: uA78M33C, L7805CV-DG:TO255P1040X460X2890-3, F.Cu at (192.0, 159.0)
- C2: value 1u -> 220u; footprint Capacitor_SMD:C_0402_1005Metric_Pad0.74x0.62mm_HandSolder -> Capacitor_THT:CP_Radial_D6.3mm_P2.50mm
- U3: value TLV70033_SOT23-5 -> L7805CV-DG; footprint Package_TO_SOT_SMD:SOT-23-5 -> L7805CV-DG:TO255P1040X460X2890-3
- moved C2 24.2 mm to (216.0, 152.5), turned to 90 degrees
- moved U3 22.7 mm to (208.0, 141.0), turned to 90 degrees
- moved U2 6.31 mm to (201.0, 141.2), turned to -90 degrees
Connections:
- C2 pad 1: +5V -> GND
- C2 pad 2: GND -> +5V
- U3 pad 1: +5V -> +12V
Routing:
- net /USART1_TX: track 55.3 -> 0.76 mm
- net /USART1_RX: track 54.2 -> 0.76 mm
- net GND: track 69.5 -> 22.7 mm
- net +3.3V: track 58.2 -> 14.5 mm, vias 2 -> 0
- net +12V: track 39.2 -> 79.7 mm
- net /USART3_TX: track 38.8 -> 0.00 mm
- net /USART3_RX: track 36.3 -> 0.00 mm
- net /USART2_TX: track 34.7 -> 0.00 mm
- net /USART2_RX: track 34.6 -> 0.00 mm
- net /SWDIO: track 33.1 -> 0.00 mm
- net /SWCLK: track 31.8 -> 0.00 mm
- net +5V: track 353.9 -> 349.9 mm
- net Net-(D4-DOUT): track 27.9 -> 29.3 mm
Other:
- board text added: "JJL v1.1"
- board text removed: "JJL v1.0"

Commit message: final
Parts:
- removed TP10, TP11, TP12, TP7, TP8, TP9: TestPoint, TestPoint:TestPoint_Pad_D3.0mm
- added J2: Conn_01x02_Pin, Connector_PinHeader_2.54mm:PinHeader_1x02_P2.54mm_Vertical, F.Cu at (200.3, 203.8)
- added J3: Conn_01x02_Pin, Connector_PinHeader_2.54mm:PinHeader_1x02_P2.54mm_Vertical, F.Cu at (171.4, 154.3)
- added J4: Conn_01x02_Pin, Connector_PinHeader_2.54mm:PinHeader_1x02_P2.54mm_Vertical, F.Cu at (229.2, 153.7)
- moved TP4 17.5 mm to (218.4, 135.0)
- moved TP15 11.3 mm to (221.9, 203.8)
- moved TP6 8.21 mm to (182.1, 135.6)
- moved U1 7.68 mm to (184.4, 185.8)
- moved C1 7.36 mm to (184.4, 179.0)
- moved U2 7.31 mm to (196.9, 147.2)
- moved D4 7.31 mm to (221.9, 157.8)
- moved D3 7.31 mm to (211.1, 139.0)
- moved J1 7.31 mm to (222.6, 178.9)
- moved D12 7.31 mm to (221.9, 195.3)
- moved D7 7.31 mm to (168.0, 176.5)
- moved D9 7.31 mm to (211.1, 176.5)
- moved D10 7.31 mm to (232.6, 176.5)
- moved D2 7.31 mm to (189.5, 139.0)
- moved D8 7.31 mm to (189.5, 176.5)
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Connections:
- U1 pad 24: unconnected-(U1-PA13-Pad24) -> /SWDIO
- U1 pad 26: /SWDIO -> unconnected-(U1-PA15-Pad26)
Routing:
- net GND: track 22.7 -> 128.7 mm, vias 9 -> 45
- net /USART1_TX: track 0.76 -> 54.0 mm
- net /USART1_RX: track 0.76 -> 53.8 mm
- net +3.3V: track 14.5 -> 55.0 mm, vias 0 -> 2
- net /SWDIO: track 0.00 -> 38.4 mm
- net /USART2_TX: track 0.00 -> 34.0 mm
- net /USART2_RX: track 0.00 -> 33.7 mm
- net /USART3_TX: track 0.00 -> 33.5 mm
- net /SWCLK: track 0.00 -> 31.5 mm
- net /USART3_RX: track 0.00 -> 31.0 mm
