File: pcb/JJL_PCB/JJL_PCB.kicad_sch (KiCad schematic)
At the start: 28 parts, among them J1 Conn_01x04_Pin, J2 Conn_01x04_Pin, J3 Conn_01x04_Pin, J4 Conn_01x04_Pin, U1 STM32G0B1KCTx, U2 L7805CV-DG, U3 TLV70033_SOT23-5

Commit message: hi
Parts:
- removed C3: 1u, Capacitor_SMD:C_0402_1005Metric_Pad0.74x0.62mm_HandSolder, symbol Device:C
- removed J2, J3, J4: Conn_01x04_Pin, Connector_PinHeader_2.54mm:PinHeader_1x04_P2.54mm_Vertical, symbol Connector:Conn_01x04_Pin
- removed U3: TLV70033_SOT23-5, Package_TO_SOT_SMD:SOT-23-5, symbol Regulator_Linear:TLV70033_SOT23-5
- added TP10, TP11, TP12, TP13, TP14, TP15, TP4, TP5, TP6, TP7, TP8, TP9: TestPoint, TestPoint:TestPoint_Pad_D3.0mm, symbol Connector:TestPoint
- added U3: L7805CV-DG, L7805CV-DG:TO255P1040X460X2890-3, symbol L7805CV-DG:L7805CV-DG
- added U4: uA78M33C, L7805CV-DG:TO255P1040X460X2890-3, symbol Regulator_Linear:uA7805
- C1: value 100n -> 1u
- C2: value 1u -> 220u; footprint Capacitor_SMD:C_0402_1005Metric_Pad0.74x0.62mm_HandSolder -> Capacitor_THT:CP_Radial_D6.3mm_P2.50mm
Connections:
- net +12V: now also U3.1 (IN), U4.1 (IN)
- net +3.3V: now also U4.3 (OUT)
- net +5V: now also C2.2, U3.3 (OUT); no longer C2.1
- net GND: now also C2.1, TP13.1, TP14.1, TP15.1, TP4.1, TP5.1, TP6.1, U3.2 (GND), U4.2 (GND); no longer C2.2
- net SWDIO: now also U1.24 (PA13); no longer U1.26 (PA15)
- net USART1_RX: now also TP8.1
- net USART1_TX: now also TP7.1
- net USART2_RX: now also TP10.1
- net USART2_TX: now also TP9.1
- net USART3_RX: now also TP12.1
- net USART3_TX: now also TP11.1
Other:
- moved on the sheet: J1, U2

Commit message: final
Parts:
- removed TP10, TP11, TP12, TP7, TP8, TP9: TestPoint, TestPoint:TestPoint_Pad_D3.0mm, symbol Connector:TestPoint
- added J2, J3, J4: Conn_01x02_Pin, Connector_PinHeader_2.54mm:PinHeader_1x02_P2.54mm_Vertical, symbol Connector:Conn_01x02_Pin
Connections:
- net USART1_RX: now also J4.1 (Pin_1)
- net USART1_TX: now also J4.2 (Pin_2)
- net USART2_RX: now also J3.1 (Pin_1)
- net USART2_TX: now also J3.2 (Pin_2)
- net USART3_RX: now also J2.1 (Pin_1)
- net USART3_TX: now also J2.2 (Pin_2)
Changed lines of the file:
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@@
     (stroke (width 0) (type default))
   )
-  (wire (pts (xy 252.73 121.92) (xy 261.62 121.92))
+  (wire (pts (xy 252.73 124.46) (xy 261.62 124.46))
     (stroke (width 0) (type default))
   )
@@
     (stroke (width 0) (type default))
   )
-  (wire (pts (xy 252.73 111.76) (xy 261.62 111.76))
+  (wire (pts (xy 252.73 114.3) (xy 261.62 114.3))
     (stroke (width 0) (type default))
   )
@@
     (stroke (width 0) (type default))
   )
-  (wire (pts (xy 252.73 101.6) (xy 261.62 101.6))
+  (wire (pts (xy 252.73 104.14) (xy 261.62 104.14))
     (stroke (width 0) (type default))
   )
@@
     (effects (font (size 1.27 1.27)) (justify left bottom))
   )
-  (label "USART1_TX" (at 252.73 101.6 180) (fields_autoplaced)
+  (label "USART1_TX" (at 252.73 104.14 180) (fields_autoplaced)
     (effects (font (size 1.27 1.27)) (justify right bottom))
   )
@@
     (effects (font (size 1.27 1.27)) (justify left bottom))
   )
-  (label "USART3_TX" (at 252.73 121.92 180) (fields_autoplaced)
+  (label "USART3_TX" (at 252.73 124.46 180) (fields_autoplaced)
     (effects (font (size 1.27 1.27)) (justify right bottom))
   )
@@
     (effects (font (size 1.27 1.27)) (justify right bottom))
   )
-  (label "USART2_TX" (at 252.73 111.76 180) (fields_autoplaced)
+  (label "USART2_TX" (at 252.73 114.3 180) (fields_autoplaced)
     (effects (font (size 1.27 1.27)) (justify right bottom))
   )
   (label "TIM2_CH1" (at 39.37 107.95 0) (fields_autoplaced)
     (effects (font (size 1.27 1.27)) (justify left bottom))
-  )
-  (symbol (lib_id "Connector:TestPoint") (at 261.62 101.6 270) (unit 1)
-    (in_bom yes) (on_board yes) (dnp no) (fields_autoplaced)
-    (property "Reference" "TP7" (at 266.7 100.965 90)
-      (effects (font (size 1.27 1.27)) (justify left))
-    )
-    (property "Value" "TestPoint" (at 266.7 103.505 90)
-      (effects (font (size 1.27 1.27)) (justify left))
-    )
-    (property "Footprint" "TestPoint:TestPoint_Pad_D3.0mm" (at 261.62 106.68 0)
-      (effects (font (size 1.27 1.27)) hide)
-    )
-    (property "Datasheet" "~" (at 261.62 106.68 0)
-      (effects (font (size 1.27 1.27)) hide)
-    )
-    (pin "1")
-    (instances
-      (project "JJL_PCB"
-        (path "/6e0934e7-8b50-43c2-9ff7-4f8375bba10f"
-          (reference "TP7") (unit 1)
-        )
-      )
-    )
   )
   (symbol (lib_id "LED:WS2812B") (at 146.05 157.48 270) (unit 1)
@@
     )
   )
-  (symbol (lib_id "Connector:TestPoint") (at 261.62 121.92 270) (unit 1)
-    (in_bom yes) (on_board yes) (dnp no) (fields_autoplaced)
-    (property "Reference" "TP11" (at 266.7 121.285 90)
-      (effects (font (size 1.27 1.27)) (justify left))
-    )
-    (property "Value" "TestPoint" (at 266.7 123.825 90)
-      (effects (font (size 1.27 1.27)) (justify left))
-    )
-    (property "Footprint" "TestPoint:TestPoint_Pad_D3.0mm" (at 261.62 127 0)
-      (effects (font (size 1.27 1.27)) hide)
-    )
-    (property "Datasheet" "~" (at 261.62 127 0)
-      (effects (font (size 1.27 1.27)) hide)
-    )
-    (pin "1")
-    (instances
-      (project "JJL_PCB"
-        (path "/6e0934e7-8b50-43c2-9ff7-4f8375bba10f"
-          (reference "TP11") (unit 1)
-        )
-      )
-    )
-  )
   (symbol (lib_id "power:+5V") (at 104.14 43.18 270) (unit 1)
     (in_bom yes) (on_board yes) (dnp no) (fields_autoplaced)
@@
         (path "/6e0934e7-8b50-43c2-9ff7-4f8375bba10f"
           (reference "#PWR032") (unit 1)
-        )
-      )
-    )
-  )
-  (symbol (lib_id "Connector:TestPoint") (at 261.62 111.76 270) (unit 1)
-    (in_bom yes) (on_board yes) (dnp no) (fields_autoplaced)
-    (property "Reference" "TP9" (at 266.7 111.125 90)
-      (effects (font (size 1.27 1.27)) (justify left))
-    )
-    (property "Value" "TestPoint" (at 266.7 113.665 90)
-      (effects (font (size 1.27 1.27)) (justify left))
-    )
-    (property "Footprint" "TestPoint:TestPoint_Pad_D3.0mm" (at 261.62 116.84 0)
-      (effects (font (size 1.27 1.27)) hide)
-    )
-    (property "Datasheet" "~" (at 261.62 116.84 0)
-      (effects (font (size 1.27 1.27)) hide)
-    )
-    (pin "1")
-    (instances
-      (project "JJL_PCB"
-        (path "/6e0934e7-8b50-43c2-9ff7-4f8375bba10f"
-          (reference "TP9") (unit 1)
         )
       )
@@
         (path "/6e0934e7-8b50-43c2-9ff7-4f8375bba10f"
           (reference "#PWR08") (unit 1)
+        )
+      )
+    )
+  )
+  (symbol (lib_id "Connector:Conn_01x02_Pin") (at 266.7 127 180) (unit 1)
+    (in_bom yes) (on_board yes) (dnp no)
+    (property "Reference" "J2" (at 275.59 127 0)
+      (effects (font (size 1.27 1.27)))
+    )
+    (property "Value" "Conn_01x02_Pin" (at 275.59 124.46 0)
+      (effects (font (size 1.27 1.27)))
+    )
+    (property "Footprint" "Connector_PinHeader_2.54mm:PinHeader_1x02_P2.54mm_Vertical" (at 266.7 127 0)
+      (effects (font (size 1.27 1.27)) hide)
+    )
+    (property "Datasheet" "~" (at 266.7 127 0)
+      (effects (font (size 1.27 1.27)) hide)
+    )
+    (pin "1")
+    (pin "2")
+    (instances
+      (project "JJL_PCB"
+        (path "/6e0934e7-8b50-43c2-9ff7-4f8375bba10f"
+          (reference "J2") (unit 1)
         )
       )
@@
     )
   )
-  (symbol (lib_id "Connector:TestPoint") (at 261.62 116.84 270) (unit 1)
-    (in_bom yes) (on_board yes) (dnp no) (fields_autoplaced)
-    (property "Reference" "TP10" (at 266.7 116.205 90)
-      (effects (font (size 1.27 1.27)) (justify left))
-    )
-    (property "Value" "TestPoint" (at 266.7 118.745 90)
-      (effects (font (size 1.27 1.27)) (justify left))
-    )
-    (property "Footprint" "TestPoint:TestPoint_Pad_D3.0mm" (at 261.62 121.92 0)
-      (effects (font (size 1.27 1.27)) hide)
-    )
-    (property "Datasheet" "~" (at 261.62 121.92 0)
-      (effects (font (size 1.27 1.27)) hide)
-    )
-    (pin "1")
-    (instances
-      (project "JJL_PCB"
-        (path "/6e0934e7-8b50-43c2-9ff7-4f8375bba10f"
-          (reference "TP10") (unit 1)
-        )
-      )
-    )
-  )
   (symbol (lib_id "LED:WS2812B") (at 74.93 142.24 270) (unit 1)
     (in_bom yes) (on_board yes) (dnp no) (fields_autoplaced)
@@
     )
   )
-  (symbol (lib_id "Connector:TestPoint") (at 261.62 106.68 270) (unit 1)
-    (in_bom yes) (on_board yes) (dnp no) (fields_autoplaced)
-    (property "Reference" "TP8" (at 266.7 106.045 90)
-      (effects (font (size 1.27 1.27)) (justify left))
-    )
-    (property "Value" "TestPoint" (at 266.7 108.585 90)
-      (effects (font (size 1.27 1.27)) (justify left))
-    )
-    (property "Footprint" "TestPoint:TestPoint_Pad_D3.0mm" (at 261.62 111.76 0)
-      (effects (font (size 1.27 1.27)) hide)
-    )
-    (property "Datasheet" "~" (at 261.62 111.76 0)
-      (effects (font (size 1.27 1.27)) hide)
-    )
-    (pin "1")
-    (instances
-      (project "JJL_PCB"
-        (path "/6e0934e7-8b50-43c2-9ff7-4f8375bba10f"
-          (reference "TP8") (unit 1)
-        )
-      )
-    )
-  )
   (symbol (lib_id "Connector:TestPoint") (at 261.62 60.96 270) (unit 1)
     (in_bom yes) (on_board yes) (dnp no) (fields_autoplaced)
@@
     )
   )
-  (symbol (lib_id "Connector:TestPoint") (at 261.62 127 270) (unit 1)
-    (in_bom yes) (on_board yes) (dnp no) (fields_autoplaced)
-    (property "Reference" "TP12" (at 266.7 126.365 90)
-      (effects (font (size 1.27 1.27)) (justify left))
-    )
-    (property "Value" "TestPoint" (at 266.7 128.905 90)
-      (effects (font (size 1.27 1.27)) (justify left))
-    )
-    (property "Footprint" "TestPoint:TestPoint_Pad_D3.0mm" (at 261.62 132.08 0)
-      (effects (font (size 1.27 1.27)) hide)
-    )
-    (property "Datasheet" "~" (at 261.62 132.08 0)
-      (effects (font (size 1.27 1.27)) hide)
-    )
-    (pin "1")
-    (instances
-      (project "JJL_PCB"
-        (path "/6e0934e7-8b50-43c2-9ff7-4f8375bba10f"
-          (reference "TP12") (unit 1)
+  (symbol (lib_id "Connector:Conn_01x02_Pin") (at 266.7 106.68 180) (unit 1)
+    (in_bom yes) (on_board yes) (dnp no)
+    (property "Reference" "J4" (at 275.59 106.68 0)
+      (effects (font (size 1.27 1.27)))
+    )
+    (property "Value" "Conn_01x02_Pin" (at 275.59 104.14 0)
+      (effects (font (size 1.27 1.27)))
+    )
+    (property "Footprint" "Connector_PinHeader_2.54mm:PinHeader_1x02_P2.54mm_Vertical" (at 266.7 106.68 0)
+      (effects (font (size 1.27 1.27)) hide)
+    )
+    (property "Datasheet" "~" (at 266.7 106.68 0)
+      (effects (font (size 1.27 1.27)) hide)
+    )
+    (pin "1")
+    (pin "2")
+    (instances
+      (project "JJL_PCB"
+        (path "/6e0934e7-8b50-43c2-9ff7-4f8375bba10f"
+          (reference "J4") (unit 1)
         )
       )
@@
         )
       )
+    )
+  )
+  (symbol (lib_id "Connector:Conn_01x02_Pin") (at 266.7 116.84 180) (unit 1)
+    (in_bom yes) (on_board yes) (dnp no)
+    (property "Reference" "J3" (at 275.59 116.84 0)
+      (effects (font (size 1.27 1.27)))
+    )
+    (property "Value" "Conn_01x02_Pin" (at 275.59 114.3 0)
+      (effects (font (size 1.27 1.27)))
+    )
+    (property "Footprint" "Connector_PinHeader_2.54mm:PinHeader_1x02_P2.54mm_Vertical" (at 266.7 116.84 0)
+      (effects (font (size 1.27 1.27)) hide)
+    )
+    (property "Datasheet" "~" (at 266.7 116.84 0)
+      (effects (font (size 1.27 1.27)) hide)
+    )
+    (pin "1")
+    (pin "2")
+    (instances
+      (project "JJL_PCB"
+        (path "/6e0934e7-8b50-43c2-9ff7-4f8375bba10f"
+          (reference "J3") (unit 1)
+        )
+      )
